Commit message: Finalized URDF file and rviz config, updated join state publisher node, successful launch test

File: my_rb1_description/urdf/my_rb1_robot.urdf (robot description, URDF)
Before this commit: robot rb1_robot, 7 links, 6 joints
Links:
- link back_caster: mass None -> 0.1; geometry collision sphere radius=0.025; visual sphere radius=0.025
- link base_link: mass None -> 23.5; geometry collision cylinder length=0.30 radius=0.25; visual cylinder length=0.30 radius=0.25
- link front_caster: mass None -> 0.1; geometry collision sphere radius=0.025; visual sphere radius=0.025
- link left_wheel: mass None -> 0.4; geometry collision cylinder length=0.02 radius=0.025; visual cylinder length=0.02 radius=0.025
- link right_wheel: mass None -> 0.4; geometry collision cylinder length=0.02 radius=0.025; visual cylinder length=0.02 radius=0.025
Joints:
- joint base_link_back_caster_joint: child (none) -> back_caster; origin (none) -> xyz=0.1 0.0 -0.15 rpy=0 0 0; parent (none) -> base_link; type  -> fixed
- joint base_link_front_caster_joint: child (none) -> front_caster; origin (none) -> xyz=-0.1 0.0 -0.15 rpy=0 0 0; parent (none) -> base_link; type  -> fixed
- joint base_link_front_laser_joint: child (none) -> front_laser; origin (none) -> xyz=0.25 0.0 0.075 rpy=3.14159265359 0 0; parent (none) -> base_link; type  -> fixed
- joint base_link_left_wheel_joint: axis (none) -> 0 1 0; child (none) -> left_wheel; origin (none) -> xyz=0.0 0.2 -0.15 rpy=0 0 0; parent (none) -> base_link; type  -> continuous
- joint base_link_plate_joint: child (none) -> base_link; origin (none) -> xyz=0 0 0.15 rpy=0 0 0; parent (none) -> base_footprint; type  -> fixed
- joint base_link_right_wheel_joint: axis (none) -> 0 1 0; child (none) -> right_wheel; origin (none) -> xyz=0.0 -0.2 -0.15 rpy=0 0 0; parent (none) -> base_link; type  -> continuous

Commit message: Added TFs to Rviz, swapped caster wheel positions, updated laser mass

File: my_rb1_description/urdf/my_rb1_robot.urdf (robot description, URDF)
Before this commit: robot rb1_robot, 7 links, 6 joints
Links:
- link front_laser: mass None -> 0.5
Joints:
- joint base_link_back_caster_joint: origin xyz=0.1 0.0 -0.15 rpy=0 0 0 -> xyz=-0.1 0.0 -0.15 rpy=0 0 0
- joint base_link_front_caster_joint: origin xyz=-0.1 0.0 -0.15 rpy=0 0 0 -> xyz=0.1 0.0 -0.15 rpy=0 0 0

Commit message: Updated laser link definition, increased rotation service speed

File: my_rb1_description/urdf/my_rb1_robot.urdf (robot description, URDF)
Before this commit: robot rb1_robot, 7 links, 6 joints
Links:
- link front_laser: mass None -> 0.5

Commit message: Aligned my_rb1_robot.urdf to reference

File: my_rb1_description/urdf/my_rb1_robot.urdf (robot description, URDF)
Before this commit: robot rb1_robot, 7 links, 6 joints
Links:
- link back_caster: mass 0.1 -> 0.5
- link base_link: mass 23.5 -> 20.5; geometry collision cylinder length=0.3 radius=0.25; visual cylinder length=0.3 radius=0.25
- link front_caster: mass 0.1 -> 0.5
- link front_laser: mass 0.5 -> None
- link left_wheel: mass 0.4 -> 1.5; geometry collision cylinder length=0.03 radius=0.025; visual cylinder length=0.03 radius=0.025
- link right_wheel: mass 0.4 -> 1.5; geometry collision cylinder length=0.03 radius=0.025; visual cylinder length=0.03 radius=0.025
Joints:
- joint base_link_back_caster_joint: origin xyz=0.1 0.0 -0.15 rpy=0 0 0 -> xyz=-0.1 0.0 -0.15 rpy=0 0 0
- joint base_link_front_caster_joint: origin xyz=-0.1 0.0 -0.15 rpy=0 0 0 -> xyz=0.1 0.0 -0.15 rpy=0 0 0
- joint base_link_front_laser_joint: origin xyz=0.25 0.0 0.075 rpy=3.14159265359 0 0 -> xyz=0.25 0 0.075 rpy=3.14 0 0
- joint base_link_left_wheel_joint: origin xyz=0.0 0.2 -0.15 rpy=0 0 0 -> xyz=0 0.2 -0.15 rpy=0 0 0
- joint base_link_right_wheel_joint: origin xyz=0.0 -0.2 -0.15 rpy=0 0 0 -> xyz=0 -0.2 -0.15 rpy=0 0 0
